File: audiograb.kicad_pcb (KiCad board)
At the start: 2 copper layers, 97 parts, among them IC1 USB2244I-AEZG-06, J1 USB_C_Receptacle_USB2.0_16P, J10 TestPoint, J11 TestPoint, J12 TestPoint, J13 TestPoint, J14 TestPoint, J15 F32Q-1A7H1-11022, J16 MEM2075-00-140-01-A, J17 691137710002, J2 SAM10346-ND, J3 Conn_02x20_Odd_Even, J4 CONMHF1-SMD-G-T, J5 CONMHF1-SMD-G-T, J6 TestPoint, J7 TestPoint, J8 TestPoint, J9 TestPoint, M1 ComputeModule5-CM5, P1 SF72S006VBAR2500, Q1 Q_PMOS_GSD, SW1 1825910-6, U1 RC7620_1104625, U10 CD4043BDR, U11 TPS22919DCKR, U12 IP4220CZ6F, U2 NX3008NBKW_115, U3 NX3008NBKW_115, U4 NX3008NBKW_115, U5 NX3008NBKW_115, U6 NX3008NBKW_115, U7 NX3008NBKW_115, U8 MAX4996LETG_

Commit message: started pcb
Parts:
- added C20: 100n, Capacitor_SMD:C_0603_1608Metric, F.Cu at (247.7, 154.0)
- added D1: D_TVS, Diode_SMD:D_0402_1005Metric, F.Cu at (261.5, 77.5)
- added J18: 3V7_in, 691137710002:691137710002, F.Cu at (274.5, 130.0)
- added J19: 3V3_in, 691137710002:691137710002, F.Cu at (251.5, 159.5)
- added J20: 5V_in, 691137710002:691137710002, F.Cu at (274.5, 152.5)
- J17: value 691137710002 -> 5V_out
- moved BT1 189.8 mm to (271.0, 39.5)
- moved CR4 167.9 mm to (32.5, 93.0), turned to 180 degrees
- moved C17 163.4 mm to (228.2, 40.5)
- moved J3 163.3 mm to (227.9, 17.0), turned to 90 degrees
- moved C18 161.7 mm to (227.3, 46.0)
- moved R2 160.8 mm to (222.7, 39.5)
- moved U1 158.8 mm to (264.6, 94.2)
- moved J5 156.7 mm to (275.0, 112.0)
- moved C19 155.3 mm to (219.8, 45.5)
- moved J4 152.6 mm to (265.0, 112.0)
- moved C4 151.2 mm to (264.5, 133.5)
- moved C6 150.4 mm to (264.5, 136.5)
- moved C8 149.6 mm to (264.5, 139.5)
- moved J2 139.2 mm to (203.9, 17.0), turned to 90 degrees
- moved IC1 134.8 mm to (89.0, 43.9)
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Connections:
- net +1V8 renamed +1V8_CM5
- net 3v3 renamed +3v3_e
- C1 pad 1: /+5V -> +5V
- C12 pad 1: +3V3 -> +3V3_CM5
- C18 pad 1: +3V3 -> +3V3_CM5
- C2 pad 1: /+5V -> +5V
- C4 pad 1: +3V8 -> VBAT_BB
- C6 pad 1: +3V8 -> VBAT_BB
- C8 pad 1: +3V8 -> VBAT_BB
- C9 pad 1: +3V3 -> +3V3_e
- CR3 pad 2: Net-(CR3-Pad2) -> /modem/UIM_CLK
- CR3 pad 5: /modem/UIM_CLK -> /modem/UIM_VCC
- CR3 pad 6: /modem/UIM_CLK -> /modem/UIM_VCC
- CR3 pad 9: Net-(CR3-Pad2) -> /modem/UIM_CLK
- CR4 pad 2: /+5V -> +5V
- D11 pad 2: +3V8 -> +3V3_CM5
- D5 pad 2: +3V3 -> +3V3_CM5
- IC1 pad 14: /usb-interface/VDD33 -> +3V3_CM5
- IC1 pad 22: /usb-interface/VDD33 -> +3V3_CM5
- IC1 pad 36: /usb-interface/VDD33 -> +3V3_CM5
- IC1 pad 6: /usb-interface/VDD33 -> +3V3_CM5
- J1 pad A4: /+5V -> +5V
- J1 pad A9: /+5V -> +5V
- J1 pad B4: /+5V -> +5V
- J1 pad B9: /+5V -> +5V
- J3 pad 1: +3V3 -> +3V3_CM5
- J3 pad 17: +3V3 -> +3V3_CM5
- M1 pad 84: +3V3 -> +3V3_CM5
- M1 pad 86: +3V3 -> +3V3_CM5
- P1 pad DSW: Net-(CR3-Pad2) -> Net-(D1-A2)
- Q1 pad 2: +3V3 -> +3V3_e
- R1 pad 2: /+5V -> +5V
- R13 pad 1: +3V8 -> +3V3_CM5
- R15 pad 1: +3V3 -> +3V3_e
- R8 pad 2: Net-(CR3-Pad2) -> Net-(D1-A2)
- U1 pad 157: +3V8 -> VBAT_BB
- U1 pad 158: +3V8 -> VBAT_BB
- U1 pad 16: +3V8 -> VBAT_BB
- U1 pad 61: +3V8 -> VBAT_BB
- U1 pad 62: +3V8 -> VBAT_BB
- U1 pad 63: +3V8 -> VBAT_BB
- U12 pad 5: /+5V -> +5V
- U5 pad 1: Net-(CR3-Pad2) -> Net-(D1-A2)
- U8 pad 14: +3V3 -> +3V3_e
- U9 pad 16: +3V3 -> +3V3_CM5
Routing:
- net /sd-interface/SD1: track 0.00 -> 8.44 mm
- net /sd-interface/SD2: track 0.00 -> 7.14 mm
- net /sd-interface/SD8: track 0.00 -> 7.09 mm
- net /sd-interface/SD3: track 0.00 -> 6.95 mm
- net /sd-interface/SD7: track 0.00 -> 6.79 mm
- net /sd-interface/SD5: track 0.00 -> 6.03 mm
Other:
- copper layers 2 -> 4

Commit message: started pcb design
Parts:
- moved J18 191.4 mm to (86.1, 96.1), turned to 0 degrees
- moved J19 190.8 mm to (71.7, 95.8)
- moved C20 186.9 mm to (71.9, 90.6)
- moved C4 186.5 mm to (83.1, 90.2), turned to 90 degrees
- moved C6 185.2 mm to (85.2, 90.2), turned to 90 degrees
- moved C8 183.9 mm to (87.3, 90.2), turned to 90 degrees
- moved J20 171.0 mm to (113.1, 96.0), turned to 0 degrees
- moved D6 165.4 mm to (244.1, 44.2), turned to 90 degrees
- moved D7 159.9 mm to (243.7, 53.9), turned to 90 degrees
- moved R8 155.5 mm to (229.4, 74.8), turned to 90 degrees
- moved C7 154.5 mm to (235.8, 84.3)
- moved C5 152.7 mm to (235.8, 82.0)
- moved C3 150.9 mm to (235.8, 79.7)
- moved CR3 149.4 mm to (244.0, 74.4), turned to 90 degrees
- moved R10 147.0 mm to (234.3, 75.0), turned to 90 degrees
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Connections:
- net /compute-module/BOOT_MODE renamed /MODEM_BOOT_MODE
- net /compute-module/Buffer_SD2 renamed /SD2
- net /compute-module/Buffer_SD3 renamed /SD3
- net /compute-module/Buffer_SD5 renamed /SD5
- net /compute-module/Buffer_SD7 renamed /SD7
- net /compute-module/GPCLK renamed /GPCLK
- net /compute-module/GPIO3 renamed /USB_INT_RESET
- net /compute-module/POWER_ON_N renamed /MODEM_POWER_ON_N
- net /compute-module/RESET_IN_N renamed /MODEM_RESET_N
- net /compute-module/R_EN_SWITCH renamed /SD_RESET_HOST
- net /compute-module/S_EN_VOUT renamed /EXT_5V_ENABLE
- net /compute-module/TX_ON renamed /MODEM_TX_ON
- net /compute-module/USB3-0-D_N renamed /USB3-0-D_N
- net /compute-module/USB3-0-D_P renamed /USB3-0-D_P
- net /compute-module/USB3-1-D_N renamed /USB3-1-D_N
- net /compute-module/USB3-1-D_P renamed /USB3-1-D_P
- net /compute-module/USBOTG_ID renamed /compute-module/USB_OTG_ID
- net /compute-module/VBUS_EN renamed /VBUS_EN
- net /modem/WAKE_ON_WWAN renamed /CM_WAKE_ON_WWAN
- net CC1 renamed /CC1
- C10 pad 1: +1V8_CM5 -> +1V8
- C12 pad 1: +3V3_CM5 -> +3V3
- D11 pad 2: +3V3_CM5 -> +3V3
- J1 pad A6: /compute-module/USB2_P -> /USB2_P
- J1 pad A7: /compute-module/USB2_N -> /USB2_N
- J1 pad B5: CC2 -> /CC2
- J1 pad B6: /compute-module/USB2_P -> /USB2_P
- J1 pad B7: /compute-module/USB2_N -> /USB2_N
- J3 pad 1: +3V3_CM5 -> +3V3
- J3 pad 17: +3V3_CM5 -> +3V3
- J3 pad 19: /compute-module/GPIO10 -> /MODEM_WAKE
- J3 pad 33: /compute-module/+1.8V -> +1V8
- M1 pad 100: /compute-module/CAM_GPIO1 -> unconnected-(M1A-CAM_GPIO1-Pad100)
- M1 pad 103: /compute-module/USB2_N -> /USB2_N
- M1 pad 105: /compute-module/USB2_P -> /USB2_P
- M1 pad 115: /compute-module/DPHY0_D0_N -> unconnected-(M1B-MIPI0_D0_N-Pad115)
- M1 pad 117: /compute-module/DPHY0_D0_P -> unconnected-(M1B-MIPI0_D0_P-Pad117)
- M1 pad 121: /compute-module/DPHY0_D1_N -> unconnected-(M1B-MIPI0_D1_N-Pad121)
- M1 pad 123: /compute-module/DPHY0_D1_P -> unconnected-(M1B-MIPI0_D1_P-Pad123)
- M1 pad 127: /compute-module/DPHY0_C_N -> unconnected-(M1B-MIPI0_C_N-Pad127)
- M1 pad 129: /compute-module/DPHY0_C_P -> unconnected-(M1B-MIPI0_C_P-Pad129)
- M1 pad 133: /compute-module/DPHY0_D2_N -> unconnected-(M1B-MIPI0_D2_N-Pad133)
- M1 pad 135: /compute-module/DPHY0_D2_P -> unconnected-(M1B-MIPI0_D2_P-Pad135)
- M1 pad 139: /compute-module/DPHY0_D3_N -> unconnected-(M1B-MIPI0_D3_N-Pad139)
- M1 pad 141: /compute-module/DPHY0_D3_P -> unconnected-(M1B-MIPI0_D3_P-Pad141)
- M1 pad 143: /compute-module/HDMI1_HOTPLUG -> unconnected-(M1B-HDMI1_HOTPLUG-Pad143)
- M1 pad 145: /compute-module/HDMI1_SDA -> unconnected-(M1B-HDMI1_SDA-Pad145)
- M1 pad 146: /compute-module/HDMI1_D2_P -> unconnected-(M1B-HDMI1_TX2_P-Pad146)
- M1 pad 147: /compute-module/HDMI1_SCL -> unconnected-(M1B-HDMI1_SCL-Pad147)
- M1 pad 148: /compute-module/HDMI1_D2_N -> unconnected-(M1B-HDMI1_TX2_N-Pad148)
- M1 pad 149: /compute-module/HDMI1_CEC -> unconnected-(M1B-HDMI1_CEC-Pad149)
- M1 pad 151: /compute-module/HDMI0_CEC -> unconnected-(M1B-HDMI0_CEC-Pad151)
- M1 pad 152: /compute-module/HDMI1_D1_P -> unconnected-(M1B-HDMI1_TX1_P-Pad152)
- M1 pad 153: /compute-module/HDMI0_HOTPLUG -> unconnected-(M1B-HDMI0_HOTPLUG-Pad153)
- M1 pad 154: /compute-module/HDMI1_D1_N -> unconnected-(M1B-HDMI1_TX1_N-Pad154)
- M1 pad 158: /compute-module/HDMI1_D0_P -> unconnected-(M1B-HDMI1_TX0_P-Pad158)
- M1 pad 160: /compute-module/HDMI1_D0_N -> unconnected-(M1B-HDMI1_TX0_N-Pad160)
- M1 pad 164: /compute-module/HDMI1_CK_P -> unconnected-(M1B-HDMI1_CLK_P-Pad164)
- M1 pad 166: /compute-module/HDMI1_CK_N -> unconnected-(M1B-HDMI1_CLK_N-Pad166)
- M1 pad 170: /compute-module/HDMI0_D2_P -> unconnected-(M1B-HDMI0_TX2_P-Pad170)
- M1 pad 172: /compute-module/HDMI0_D2_N -> unconnected-(M1B-HDMI0_TX2_N-Pad172)
- M1 pad 175: /compute-module/DPHY1_D0_N -> unconnected-(M1B-MIPI1_D0_N-Pad175)
- M1 pad 176: /compute-module/HDMI0_D1_P -> unconnected-(M1B-HDMI0_TX1_P-Pad176)
- M1 pad 177: /compute-module/DPHY1_D0_P -> unconnected-(M1B-MIPI1_D0_P-Pad177)
- M1 pad 178: /compute-module/HDMI0_D1_N -> unconnected-(M1B-HDMI0_TX1_N-Pad178)
- M1 pad 181: /compute-module/DPHY1_D1_N -> unconnected-(M1B-MIPI1_D1_N-Pad181)
- M1 pad 182: /compute-module/HDMI0_D0_P -> unconnected-(M1B-HDMI0_TX0_P-Pad182)
- M1 pad 183: /compute-module/DPHY1_D1_P -> unconnected-(M1B-MIPI1_D1_P-Pad183)
- M1 pad 184: /compute-module/HDMI0_D0_N -> unconnected-(M1B-HDMI0_TX0_N-Pad184)
- M1 pad 187: /compute-module/DPHY1_C_N -> unconnected-(M1B-MIPI1_C_N-Pad187)
- M1 pad 188: /compute-module/HDMI0_CK_P -> unconnected-(M1B-HDMI0_CLK_P-Pad188)
- M1 pad 189: /compute-module/DPHY1_C_P -> unconnected-(M1B-MIPI1_C_P-Pad189)
- M1 pad 190: /compute-module/HDMI0_CK_N -> unconnected-(M1B-HDMI0_CLK_N-Pad190)
- M1 pad 193: /compute-module/DPHY1_D2_N -> unconnected-(M1B-MIPI1_D2_N-Pad193)
- M1 pad 194: /compute-module/DPHY1_D3_N -> unconnected-(M1B-MIPI1_D3_N-Pad194)
- M1 pad 195: /compute-module/DPHY1_D2_P -> unconnected-(M1B-MIPI1_D2_P-Pad195)
- M1 pad 196: /compute-module/DPHY1_D3_P -> unconnected-(M1B-MIPI1_D3_P-Pad196)
- M1 pad 199: /compute-module/HDMI0_SDA -> unconnected-(M1B-HDMI0_SDA-Pad199)
- M1 pad 200: /compute-module/HDMI0_SCL -> unconnected-(M1B-HDMI0_SCL-Pad200)
- M1 pad 36: /compute-module/ID_SD -> unconnected-(M1A-ID_SD-Pad36)
- M1 pad 37: /compute-module/R_SWITCH -> /SD_SWITCH_ENABLE
- M1 pad 39: /compute-module/R_EN_VOUT -> /SD_SET_HOST
- M1 pad 44: /compute-module/WAKE -> /MODEM_WAKE
- M1 pad 45: /compute-module/S_SWITCH -> /SD_SWITCH_DISABLE
- M1 pad 49: /compute-module/S_EN_SWITCH -> /EXT_5V_DISABLE
- M1 pad 80: /compute-module/SCL0 -> unconnected-(M1A-SCL0-Pad80)
- M1 pad 82: /compute-module/SDA0 -> unconnected-(M1A-SDA0-Pad82)
- M1 pad 96: CC2 -> /CC2
- M1 pad 97: /compute-module/CAM_GPIO0 -> unconnected-(M1A-CAM_GPIO0-Pad97)
- R1 pad 1: GND -> +5V
- R1 pad 2: +5V -> GND
- R13 pad 1: +3V3_CM5 -> +3V3
- R15 pad 2: Net-(U10-Q3) -> Net-(U10-Q1)
- R16 pad 1: Net-(U10-Q3) -> Net-(U10-Q1)
- R3 pad 1: /compute-module/WAKE -> /modem/WAKE
- U10 pad 11: /compute-module/R_SWITCH -> /SD_SWITCH_ENABLE
- U10 pad 12: /compute-module/S_SWITCH -> /SD_SWITCH_DISABLE
- U10 pad 14: /compute-module/S_EN_SWITCH -> /SD_SET_HOST
- U10 pad 2: unconnected-(U10-Q1-Pad2) -> Net-(U10-Q1)
- U10 pad 3: unconnected-(U10-R1-Pad3) -> /SD_SWITCH_ENABLE
- U10 pad 4: unconnected-(U10-S1-Pad4) -> /SD_SWITCH_DISABLE
- U10 pad 7: /compute-module/R_EN_VOUT -> /EXT_5V_DISABLE
- U12 pad 1: /compute-module/USB2_N -> /USB2_P
- U12 pad 3: /compute-module/USB2_P -> /CC2
- U12 pad 6: CC2 -> /USB2_N
- U9 pad 1: +1V8_CM5 -> +1V8
- U9 pad 16: +3V3_CM5 -> +3V3
- U9 pad 2: +1V8_CM5 -> +1V8
- U9 pad 3: +1V8_CM5 -> +1V8
Routing:
- net +5V: track 0.00 -> 35.8 mm
- net /compute-module/GPIO26: track 0.00 -> 28.0 mm
- net /compute-module/GPIO19: track 0.00 -> 25.5 mm
- net Net-(J16-DAT2): track 0.00 -> 23.5 mm, vias 0 -> 2
- net /compute-module/GPIO2: track 0.00 -> 22.2 mm
- net GND: track 0.00 -> 21.2 mm, vias 0 -> 3
- net Net-(J16-CD/DAT3): track 0.00 -> 20.8 mm, vias 0 -> 2
- net Net-(J16-CMD): track 0.00 -> 18.5 mm, vias 0 -> 2
- net /compute-module/GPIO12: track 0.00 -> 17.4 mm
- net +3v3_e: track 0.00 -> 16.8 mm
- net /compute-module/GPIO17: track 0.00 -> 13.6 mm, vias 0 -> 2
- net /compute-module/GPIO11: track 0.00 -> 13.3 mm, vias 0 -> 2
- net /compute-module/ID_SC: track 0.00 -> 13.1 mm
- net Net-(J16-DAT1): track 0.00 -> 13.0 mm, vias 0 -> 2
- net /compute-module/GPIO27: track 0.00 -> 12.9 mm, vias 0 -> 2
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
Commit message: work pcb about 70 percent
Parts:
- removed J20: 5V_in, 691137710002:691137710002
- added C21: 4.7uF, Capacitor_SMD:C_0603_1608Metric, F.Cu at (117.9, 47.7)
- added C22: 4.7uF, Capacitor_SMD:C_0603_1608Metric, F.Cu at (117.2, 58.7)
- added C23: 4.7uF, Capacitor_SMD:C_0603_1608Metric, F.Cu at (121.7, 50.7)
- added C24: 4.7uF, Capacitor_SMD:C_0603_1608Metric, F.Cu at (112.7, 57.9)
- IC1: footprint USB2244I-AEZG-06:QFN50P600X600X90-37N-D -> Package_DFN_QFN:QFN-36-1EP_6x6mm_P0.5mm_EP4.1x4.1mm_ThermalVias
- J10, J11, J12, J13, J14, J6, J7, J8, J9, TP1, TP13, TP14, TP15, TP16, TP17, TP18, TP19, TP3, TP4, TP5, TP6: footprint TestPoint:TestPoint_Loop_D2.50mm_Drill1.85mm -> TestPoint:TestPoint_Loop_D2.60mm_Drill1.6mm_Beaded
- TP10, TP11, TP12, TP7, TP8, TP9: footprint TestPoint:TestPoint_Loop_D2.50mm_Drill1.85mm -> TestPoint:TestPoint_Pad_D1.0mm
- moved J11 253.6 mm to (170.2, -29.7)
- moved TP3 250.6 mm to (175.3, -29.7)
- moved TP2 248.4 mm to (180.6, -29.5)
- moved J8 245.2 mm to (165.2, -19.6)
- moved J7 244.8 mm to (165.2, -24.6)
- moved J6 244.2 mm to (165.1, -29.5)
- moved J14 237.8 mm to (170.2, -14.6)
- moved J13 237.4 mm to (170.2, -19.6)
- moved J12 237.1 mm to (170.2, -24.6)
- moved J10 229.1 mm to (165.2, -9.50)
- moved J9 228.8 mm to (165.2, -14.6)
- moved TP13 226.0 mm to (146.8, -35.0)
- moved TP1 221.4 mm to (170.2, -9.50)
- moved TP19 210.7 mm to (151.9, -24.9)
- moved TP17 210.0 mm to (151.9, -35.0)
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Connections:
- C13 pad 1: +3v3_e -> +3V3
- C20 pad 1: +3V3_e -> +3V3
- C9 pad 1: +3V3_e -> +3V3
- J19 pad 1: +3V3_e -> +3V3
- J3 pad 19: /MODEM_WAKE -> unconnected-(J3-Pin_19-Pad19)
- J3 pad 31: /compute-module/GPIO_VREF -> +3V3_CM5
- M1 pad 78: /compute-module/GPIO_VREF -> +3V3_CM5
- Q1 pad 2: +3V3_e -> +3V3
- R11 pad 1: /CM_WAKE_ON_WWAN -> /modem/WAKE_ON_WWAN
- R15 pad 1: +3V3_e -> +3V3
- U1 pad 110: /CM_WAKE_ON_WWAN -> /modem/WAKE_ON_WWAN
- U10 pad 16: +3v3_e -> +3V3
- U10 pad 5: +3v3_e -> +3V3
- U6 pad 1: /CM_WAKE_ON_WWAN -> /modem/WAKE_ON_WWAN
- U8 pad 14: +3V3_e -> +3V3
Routing:
- net /SD7: track 0.00 -> 106.5 mm
- net /SD3: track 0.00 -> 104.5 mm
- net /SD5: track 0.00 -> 100.1 mm
- net /SD2: track 0.00 -> 91.9 mm
- net /USB3-0-D_P: track 0.00 -> 70.9 mm, vias 0 -> 2
- net /USB3-0-D_N: track 0.00 -> 69.4 mm, vias 0 -> 2
- net Net-(U10-Q3): track 3.44 -> 55.3 mm, vias 0 -> 2
- net Net-(U10-Q4): track 4.37 -> 56.2 mm, vias 0 -> 2
- net /compute-module/EEPROM_nWP: track 0.00 -> 51.7 mm, vias 0 -> 1
- net Net-(U10-Q1): track 2.00 -> 51.6 mm, vias 0 -> 1
- net /SD_SET_HOST: track 0.00 -> 38.3 mm
- net /compute-module/nRPIBOOT: track 0.00 -> 37.5 mm, vias 0 -> 1
- net /sd-interface/SD-pin3: track 0.00 -> 33.1 mm, vias 0 -> 2
- net /modem/UIM_VCC: track 0.00 -> 32.7 mm, vias 0 -> 2
- net /compute-module/PWR_BUT: track 0.00 -> 32.0 mm, vias 0 -> 2
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Other:
- board text added: "PWR CM"

Commit message: more pcb
Parts:
- J10, J11, J12, J13, J14, J6, J7, J8, J9, TP1, TP3, TP4: footprint TestPoint:TestPoint_Loop_D2.60mm_Drill1.6mm_Beaded -> TestPoint:TestPoint_Loop_D2.50mm_Drill1.0mm
- TP2: footprint TestPoint:TestPoint_Loop_D2.50mm_Drill1.85mm -> TestPoint:TestPoint_Loop_D2.50mm_Drill1.0mm
- TP5, TP6: footprint TestPoint:TestPoint_Loop_D2.60mm_Drill1.6mm_Beaded -> TestPoint:TestPoint_Pad_D1.5mm; moved to B.Cu
- moved TP17 84.5 mm to (117.1, 42.1)
- moved J11 81.3 mm to (202.2, 45.1)
- moved J12 81.0 mm to (206.1, 48.0)
- moved TP13 77.4 mm to (107.9, 31.9)
- moved J13 77.2 mm to (202.1, 50.7)
- moved J14 76.5 mm to (206.2, 53.0)
- moved TP19 73.1 mm to (123.3, 42.4)
- moved TP2 71.8 mm to (201.8, 39.1)
- moved TP6 69.4 mm to (239.4, 12.1), turned to 180 degrees
- moved TP3 67.1 mm to (211.1, 27.1)
- moved J7 66.2 mm to (205.9, 27.6)
- moved J9 65.9 mm to (205.8, 37.4)
- moved J8 65.7 mm to (205.3, 32.5)
- moved J6 65.5 mm to (202.7, 24.1)
- moved TP5 65.5 mm to (230.5, 15.6), turned to 180 degrees
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Routing:
- net /GPCLK: track 8.55 -> 91.4 mm
- net /USB3-1-D_N: track 0.00 -> 60.7 mm, vias 0 -> 2
- net /USB3-1-D_P: track 0.00 -> 59.6 mm, vias 0 -> 2
- net /modem/UIM_SIM_DET: track 0.00 -> 58.3 mm, vias 0 -> 2
- net Net-(U10-Q2): track 0.00 -> 55.3 mm, vias 0 -> 2
- net /USB_INT_RESET: track 4.05 -> 59.3 mm
- net /modem/1V8_BOOT_MODE: track 0.00 -> 53.8 mm, vias 0 -> 2
- net /modem/1V8_POWER_ON_N: track 0.00 -> 51.9 mm, vias 0 -> 2
- net /modem/UIM_DATA: track 17.2 -> 68.2 mm
- net /modem/UIM_CLK: track 18.0 -> 62.1 mm, vias 3 -> 4
- net /modem/UIM_RESET_N: track 18.0 -> 59.6 mm, vias 3 -> 4
- net /modem/UIM_VCC: track 32.7 -> 72.5 mm, vias 2 -> 4
- net /SD_SWITCH_ENABLE: track 17.2 -> 52.7 mm, vias 0 -> 4
- net /SD_SWITCH_DISABLE: track 16.0 -> 50.1 mm, vias 0 -> 4
- net /modem/1V8_TX_ON: track 2.14 -> 35.5 mm, vias 0 -> 2
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Other:
- board outline added: 166.6 x 68.9 mm
