File: sch/power-suply.kicad_sch (KiCad schematic)
At the start: 38 parts, among them J5 12V_in, Q2 DMT6007LFG-7, U1 LMR51450SDRRR, U2 LM74700QDBVTQ1, U3 LMR51450SDRRR

Commit message: partnumber, manufaturerer and description cleanup completed
Parts:
- D2: footprint 0402ESDA-MLP1:ESD_0402ESDA-MLP1 -> Diode_SMD:D_0402_1005Metric
- J5: Description_1 2 Position Wire to Board Terminal Block Horizontal with Boa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 -> (none); MF Würth Elektronik -> (none); MP 691137710002 -> (none); MPN (none) -> 691137710002; Manufacturer (none) -> Würth Elektronik
- U1, U3: Description_1 36-V, 5-A synchronous buck converter -> (none); MANUFACTURER Texas Instruments -> (none); MP LMR51450SDRRR -> (none); MPN (none) -> LMR51450SDRRR; Manufacturer (none) -> Texas Instruments
- U2: Description_1 3.2-V to 65-V, 80-uA IQ automotive ideal diode controller -> (none); MANUFACTURER Texas Instruments -> (none); MP LM74700QDBVTQ1 -> (none); MPN (none) -> LM74700QDBVTQ1; Manufacturer (none) -> Texas Instruments
Changed lines of the file:
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@@
 			)
 		)
-		(property "Description" ""
+		(property "Description" "36-V, 5-A synchronous buck converter"
 			(at 175.26 36.83 0)
 			(effects
@@
 			)
 		)
-		(property "MP" "LMR51450SDRRR"
+		(property "MPN" "LMR51450SDRRR"
 			(at 175.26 36.83 0)
 			(effects
@@
 			)
 		)
-		(property "Description_1" "36-V, 5-A synchronous buck converter"
-			(at 175.26 36.83 0)
-			(effects
-				(font
-					(size 1.27 1.27)
-				)
-				(justify bottom)
-				(hide yes)
-			)
-		)
 		(property "Availability" "In Stock"
 			(at 175.26 36.83 0)
@@
 			)
 		)
-		(property "MANUFACTURER" "Texas Instruments"
+		(property "Manufacturer" "Texas Instruments"
 			(at 175.26 36.83 0)
 			(effects
@@
 			)
 		)
-		(property "Description" "12V power in"
+		(property "Description" "2 Position Wire to Board Terminal Block Horizontal with Board 0.197 (5.00mm) Through Hole"
 			(at 16.51 26.67 0)
 			(effects
@@
 			)
 		)
-		(property "MF" "Würth Elektronik"
-			(at 16.51 26.67 0)
-			(effects
-				(font
-					(size 1.27 1.27)
-				)
-				(justify bottom)
-				(hide yes)
-			)
-		)
-		(property "Description_1" "2 Position Wire to Board Terminal Block Horizontal with Board 0.197 (5.00mm) Through Hole"
+		(property "Manufacturer" "Würth Elektronik"
 			(at 16.51 26.67 0)
 			(effects
@@
 			)
 		)
-		(property "MP" "691137710002"
+		(property "MPN" "691137710002"
 			(at 16.51 26.67 0)
 			(effects
@@
 			)
 		)
-		(property "Description" ""
+		(property "Description" "3.2-V to 65-V, 80-uA IQ automotive ideal diode controller"
 			(at 63.5 60.96 0)
 			(effects
@@
 			)
 		)
-		(property "MP" "LM74700QDBVTQ1"
-			(at 63.5 60.96 0)
-			(effects
-				(font
-					(size 1.27 1.27)
-				)
-				(justify bottom)
-				(hide yes)
-			)
-		)
-		(property "Description_1" "3.2-V to 65-V, 80-uA IQ automotive ideal diode controller"
+		(property "MPN" "LM74700QDBVTQ1"
 			(at 63.5 60.96 0)
 			(effects
@@
 			)
 		)
-		(property "MANUFACTURER" "Texas Instruments"
+		(property "Manufacturer" "Texas Instruments"
 			(at 63.5 60.96 0)
 			(effects
@@
 			)
 		)
-		(property "Footprint" "0402ESDA-MLP1:ESD_0402ESDA-MLP1"
+		(property "Footprint" "Diode_SMD:D_0402_1005Metric"
 			(at 39.37 31.75 0)
 			(effects
@@
 			)
 		)
-		(property "Description" ""
+		(property "Description" "36-V, 5-A synchronous buck converter"
 			(at 176.53 99.06 0)
 			(effects
@@
 			)
 		)
-		(property "MP" "LMR51450SDRRR"
+		(property "MPN" "LMR51450SDRRR"
 			(at 176.53 99.06 0)
 			(effects
@@
 			)
 		)
-		(property "Description_1" "36-V, 5-A synchronous buck converter"
-			(at 176.53 99.06 0)
-			(effects
-				(font
-					(size 1.27 1.27)
-				)
-				(justify bottom)
-				(hide yes)
-			)
-		)
 		(property "Availability" "In Stock"
 			(at 176.53 99.06 0)
@@
 			)
 		)
-		(property "MANUFACTURER" "Texas Instruments"
+		(property "Manufacturer" "Texas Instruments"
 			(at 176.53 99.06 0)
 			(effects
